Commit message: Update control

File: src/robotmodel/urdf/eros (bckup).urdf (robot description, URDF)
Before this commit: robot EROS, 40 links, 39 joints
Joints:
- removed joint kaki_kanan_kiri
- added joint kaki_kiri_eof: type fixed, parent telapak_kaki_kiri, child telapak_kaki_kiri_eof, origin xyz=0 0.0 -0.055, axis 0 1 0, limit lower=-3.14 upper=3.14 effort=300 velocity=0.1
- joint bahu_kanan_pitch: axis 0 1 0 -> 0 -1 0
- joint bahu_kiri_pitch: axis 0 1 0 -> 0 -1 0
- joint bahu_kiri_roll: axis 1 0 0 -> -1 0 0
- joint engkle_kanan_roll: axis 1 0 0 -> -1 0 0
- joint hip_kanan_pitch: axis 0 1 0 -> 0 -1 0
- joint hip_kanan_yaw: axis 0 0 1 -> 0 0 -1
- joint hip_kiri_pitch: axis 0 1 0 -> 0 -1 0
- joint hip_kiri_roll: axis 1 0 0 -> -1 0 0
- joint hip_kiri_yaw: axis 0 0 1 -> 0 0 -1
- joint lutut_kiri_roll: axis 1 0 0 -> -1 0 0
- joint siku_kanan_yaw: axis 0 0 1 -> 0 0 -1
- joint siku_kiri_yaw: axis 0 0 1 -> 0 0 -1
